Commit message: Import ur10e description

File: urdf/ur10e_hande.urdf (robot description, URDF)
Before this commit: robot ur10e_robot, 18 links, 17 joints
Links:
- link base_link_inertia: geometry collision mesh filename=package://robotiq_hande_description/meshes/ur10e/collision/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; visual mesh filename=meshes/ur10e/visual/base.dae
- link forearm_link: geometry collision mesh filename=package://robotiq_hande_description/meshes/ur10e/collision/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; visual mesh filename=package://robotiq_hande_description/meshes/ur10e/visual/for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
- link shoulder_link: geometry collision mesh filename=package://robotiq_hande_description/meshes/ur10e/collision/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; visual mesh filename=package://robotiq_hande_description/meshes/ur10e/visual/sho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
- link upper_arm_link: geometry collision mesh filename=package://robotiq_hande_description/meshes/ur10e/collision/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; visual mesh filename=package://robotiq_hande_description/meshes/ur10e/visual/upp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
- link wrist_1_link: geometry collision mesh filename=package://robotiq_hande_description/meshes/ur10e/collision/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; visual mesh filename=package://robotiq_hande_description/meshes/ur10e/visual/wri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
- link wrist_2_link: geometry collision mesh filename=package://robotiq_hande_description/meshes/ur10e/collision/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; visual mesh filename=package://robotiq_hande_description/meshes/ur10e/visual/wri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
- link wrist_3_link: geometry collision mesh filename=package://robotiq_hande_description/meshes/ur10e/collision/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; visual mesh filename=package://robotiq_hande_description/meshes/ur10e/visual/wri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
