Commit message: update gripper

File: urdf/robotiq_hande_gripper.xacro (robot description, xacro)
@@ -65,28 +65,9 @@
     </joint>
     <link name="${prefix}robotiq_hande_left_finger">
-      <inertial>
-        <origin rpy="0 0 0" xyz="0 0 0"/>
-        <mass value="0.03804"/>
-        <inertia ixx="1E-9" ixy="0.0" ixz="0.0" iyy="1E-9" iyz="0.0" izz="1E-9"/>
-      </inertial>
-      <collision>
-        <origin rpy="0 0 3.1415926" xyz="0 0 0"/>
-        <geometry>
-          <mesh filename="package://robotiq_hande_description/meshes/finger_collision.dae" scale="1.0 1.0 1.0"/>
-        </geometry>
-      </collision>
-      <visual>
+      <inertial>ros2 run ur_robot_driver tool_communication.py --ros-args -p robot_ip:=10.0.0.155
         <origin rpy="1.570796 0 3.1415926" xyz="0 0 0"/>
         <geometry>
           <mesh filename="package://robotiq_hande_description/meshes/finger.dae" scale="1.0 1.0 1.0"/>
-        </geometry>
-        <material name="Grey"/>
-      </visual>
-    </link>
-    <joint name="${prefix}robotiq_hande_right_finger_joint" type="prismatic">
-      <origin rpy="0 0 0" xyz="0 0.025 0.0345"/>
-      <parent link="${prefix}robotiq_hande_link"/>
-      <child link="${prefix}robotiq_hande_right_finger"/>
-      <axis xyz="0 -1 0"/>
+        </geometry>ros2 run ur_robot_driver tool_communication.py --ros-args -p robot_ip:=10.0.0.155
       <limit effort="130" lower="0" upper="0.025" velocity="0.15"/>
       <mimic joint="${prefix}robotiq_hande_left_finger_joint" multiplier="1" offset="0"/>

Commit message: update mesh

File: urdf/robotiq_hande_gripper.xacro (robot description, xacro)
@@ -65,9 +65,28 @@
     </joint>
     <link name="${prefix}robotiq_hande_left_finger">
-      <inertial>ros2 run ur_robot_driver tool_communication.py --ros-args -p robot_ip:=10.0.0.155
+      <inertial>
+        <origin rpy="0 0 0" xyz="0 0 0"/>
+        <mass value="0.03804"/>
+        <inertia ixx="1E-9" ixy="0.0" ixz="0.0" iyy="1E-9" iyz="0.0" izz="1E-9"/>
+      </inertial>
+      <visual>
         <origin rpy="1.570796 0 3.1415926" xyz="0 0 0"/>
         <geometry>
           <mesh filename="package://robotiq_hande_description/meshes/finger.dae" scale="1.0 1.0 1.0"/>
-        </geometry>ros2 run ur_robot_driver tool_communication.py --ros-args -p robot_ip:=10.0.0.155
+        </geometry>
+        <material name="Grey"/>
+      </visual>
+      <collision>
+        <origin rpy="0 0 0" xyz="0 0 0"/>
+        <geometry>
+          <mesh filename="package://robotiq_hande_description/meshes/finger_collision.dae" scale="1.0 1.0 1.0"/>
+        </geometry>
+      </collision>
+    </link>
+    <joint name="${prefix}robotiq_hande_right_finger_joint" type="prismatic">
+      <origin rpy="0 0 0" xyz="0 0.025 0.0345"/>
+      <parent link="${prefix}robotiq_hande_link"/>
+      <child link="${prefix}robotiq_hande_right_finger"/>
+      <axis xyz="0 -1 0"/>
       <limit effort="130" lower="0" upper="0.025" velocity="0.15"/>
       <mimic joint="${prefix}robotiq_hande_left_finger_joint" multiplier="1" offset="0"/>
